File: base_plate/base_plate.brd (EAGLE design)
At the start: 60.5 x 69.4 mm, 7 parts

Commit message: tweaked base plate and exported to dxf
Parts:
- moved E$1 26.9 mm to (212.1, 189.2)
- moved E$3 21.6 mm to (241.0, 189.2)
- moved E$4 16.5 mm to (241.0, 143.5)
- moved E$5 11.4 mm to (241.0, 97.8)
- moved E$2 10.9 mm to (212.1, 142.2)
- moved E$6 6.35 mm to (241.0, 52.1)
- moved E$7 2.54 mm to (139.7, 10.2)
Other:
- board size 60.5 x 69.4 mm -> 341.6 x 201.9 mm
